Commit message: fix spelling error

File: src/urdf/bigbot_physical.urdf.xacro (robot description, xacro)
@@ -2,5 +2,5 @@
 <robot name="zbig" xmlns:xacro="http://ros.org/wiki/xacro">
   <link name="base_footprint"></link>
-  <joint name="base_footrint_joint" type="fixed">
+  <joint name="base_footprint_joint" type="fixed">
     <parent link="base_footprint"/>
     <child link="base_link" />
